File: PCB/Pocket lightning detector.kicad_sch (KiCad schematic)
At the start: 65 parts, among them J1 USB_C_Receptacle_USB2.0_16P, J2 Conn_01x02_Pin, Q1 FS8205A, Q2 SS8550, U1 ESP32-C3-MINI-1-N4, U2 AP2112K-3.3, U3 USBLC6-2SC6, U4 AS3935, U5 TP4056-42-ESOP8, U6 DW01A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

Commit message: Fixing PCB
Parts:
- C1: value 4uF -> 100nF
- C2: value 4uF -> 4.7uF
- C3, C4: value 4.7uF -> 10uF
- C7, C8: value TBD -> 10pF
- R4: value TBD -> NC
- Y1: value Crystal -> 32.768kHz, 7pF
Changed lines of the file:
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@@
 			)
 		)
-		(property "Value" "TBD"
+		(property "Value" "NC"
 			(at 35.56 39.37 90)
 			(effects
@@
 			)
 		)
-		(property "Value" "TBD"
+		(property "Value" "10pF"
 			(at 46.482 58.42 0)
 			(effects
@@
 			)
 		)
-		(property "Value" "Crystal"
+		(property "Value" "32.768kHz, 7pF"
 			(at 35.56 48.26 0)
 			(effects
@@
 			)
 		)
-		(property "Value" "4uF"
+		(property "Value" "100nF"
 			(at 151.13 97.7899 0)
 			(effects
@@
 			)
 		)
-		(property "Value" "4.7uF"
+		(property "Value" "10uF"
 			(at 24.13 165.0999 0)
 			(effects
@@
 			)
 		)
-		(property "Value" "4.7uF"
+		(property "Value" "10uF"
 			(at 57.15 165.0999 0)
 			(effects
@@
 			)
 		)
-		(property "Value" "4uF"
+		(property "Value" "4.7uF"
 			(at 165.1 97.7899 0)
 			(effects
@@
 			)
 		)
-		(property "Value" "TBD"
+		(property "Value" "10pF"
 			(at 30.48 58.4199 0)
 			(effects
